File: hardware/horae.sch (KiCad schematic (older format))
At the start: 60 parts, among them J1 Conn_PIC_ICSP_ICD, J2 USB_B_Micro, Q1 BC817, Q2 BC817, Q3 BC817, Q4 BC817, Q5 BC817, Q6 BC817, SW1 SW_DIP_x02, SW2 SW_DIP_x02, SW3 SW_DIP_x02, SW4 SW_DIP_x02, U1 ATmega328P-AU, U2 DS3231M, U3 MAX803SEXRT, X1 XTAL

Commit message: finish pcb and add horae.c
Parts:
- removed Q6: BC817, Package_TO_SOT_SMD:SOT-23, symbol Transistor_BJT:BC817
- removed R16: R, symbol Device:R
- removed SW1, SW2, SW3, SW4: SW_DIP_x02, symbol Switch:SW_DIP_x02
- added SW1, SW2, SW3, SW4: SW_Push, Button_Switch_SMD:SW_Push_1P1T-SH_NO_CK_KMR2xxG, symbol Switch:SW_Push
- C1, C2, C3, C4, C5, C7: footprint (none) -> Capacitor_SMD:C_0201_0603Metric
- C6: footprint (none) -> Capacitor_SMD:CP_Elec_3x5.3
- D1, D10, D11, D12, D13, D14, D15, D16, D17, D18, D19, D2, D20, D3, D4, D5, D6, D7, D8, D9: footprint (none) -> LED_SMD:LED-APA102-2020
- J1: footprint (none) -> Connector_PinHeader_2.54mm:PinHeader_1x06_P2.54mm_Horizontal
- J2: footprint (none) -> Connector_USB:USB_Micro-B_Amphenol_10103594-0001LF_Horizontal
- R1, R10, R11, R12, R13, R14, R15, R2, R3, R4, R5, R6, R7, R8, R9: footprint (none) -> Resistor_SMD:R_0201_0603Metric
- U3: footprint SOT65P210X110-3N -> m803:SOT65P210X110-3N
- X1: footprint (none) -> xtal:XTAL3215
Connections:
- wire segments 153 -> 151
